Commit message: modular xacro urdf files

File: src/robot_description/urdf/robot.urdf.xacro (robot description, xacro)
@@ -1,69 +1,5 @@
 <?xml version="1.0"?>
 <robot name="robot" xmlns:xacro="http://www.ros.org/wiki/xacro" >
-  <xacro:property name="base_length" value="0.6" />
-  <xacro:property name="base_width" value="0.4" />
-  <xacro:property name="base_height" value="0.2" />
-  <xacro:property name="wheel_radius" value="0.1" />
-  <xacro:property name="wheel_length" value="0.05" />
-  <material name="blue">
-    <color rgba="0 0 0.5 1" />
-  </material>
-  <material name="grey">
-    <color rgba="0.5 0.5 0.5 1"/>
-  </material>
-  <link name="base_footprint_link" />
-  <joint name="base_joint" type="fixed">
-    <parent link="base_footprint_link" />
-    <child link="base_link" />
-    <origin xyz="0 0 ${wheel_radius}" rpy="0 0 0" />
-  </joint>
-  <link name="base_link">
-    <visual>
-      <geometry>
-        <box size="${base_length} ${base_width} ${base_height}" />
-      </geometry>
-      <origin xyz="0 0 ${base_height / 2}" rpy="0 0 0" />
-      <material name="blue" />
-    </visual>
-  </link>
-  <xacro:macro name="wheel_link" params="prefix">
-    <link name="${prefix}_wheel_link">
-      <visual>
-        <geometry>
-          <cylinder radius="${wheel_radius}" length="${wheel_length}" />
-        </geometry>
-        <origin xyz="0 0 0" rpy="${pi / 2.0} 0 0" />
-        <material name="grey" />
-      </visual>
-    </link>
-  </xacro:macro>
-  <xacro:wheel_link prefix="right" />
-  <joint name="base_right_wheel_joint" type="continuous">
-    <parent link="base_link" />
-    <child link="right_wheel_link" />
-    <origin xyz="${-base_length / 4} ${-base_width / 2 - wheel_length / 2} 0" rpy="0 0 0" />
-    <axis xyz="0 1 0" />
-  </joint>
-  <xacro:wheel_link prefix="left" />
-  <joint name="base_left_wheel_joint" type="continuous">
-    <parent link="base_link" />
-    <child link="left_wheel_link" />
-    <origin xyz="${-base_length / 4} ${base_width / 2 + wheel_length / 2} 0" rpy="0 0 0" />
-    <axis xyz="0 1 0" />
-  </joint>
-  <link name="caster_wheel_link">
-    <visual>
-      <geometry>
-        <sphere radius="${wheel_radius / 2}" />
-      </geometry>
-      <origin xyz="0 0 0" rpy="0 0 0" />
-      <material name="grey" />
-    </visual>
-  </link>
-  <joint name="base_caster_wheel_joint" type="fixed">
-    <parent link="base_link" />
-    <child link="caster_wheel_link" />
-    <origin xyz="${base_length / 3.0} 0 ${-wheel_radius / 2}" rpy="0 0 0" />
-    <axis xyz="0 0 0" />
-  </joint>
+  <xacro:include filename="common_properties.xacro" />
+  <xacro:include filename="mobile_base.xacro" />
 </robot>
