Commit message: inertia xacro

File: src/robot_description/urdf/common_properties.xacro (robot description, xacro)
@@ -7,3 +7,12 @@
     <color rgba="0.5 0.5 0.5 1"/>
   </material>
+  <xacro:xacro name="box_inertia" params="m x y z o_xyz o_rpy">
+    <inertial>
+      <mass value="${m}" />
+      <origin xyz="${o_xyz}" rpy="${o_rpy}"/>
+      <inertia  ixx="${(m/12) * (y*y + z*z)}"  ixy="0" ixz="0"
+                iyy="${(m/12) * (x*x + z*z)}"  iyz="0"
+                izz="${(m/12) * (y*y + y*y)}" />
+    </inertial>
+  </xacro:xacro>
 </robot>

Commit message: inertia xacro macro include and ammend

File: src/robot_description/urdf/common_properties.xacro (robot description, xacro)
@@ -7,5 +7,5 @@
     <color rgba="0.5 0.5 0.5 1"/>
   </material>
-  <xacro:xacro name="box_inertia" params="m x y z o_xyz o_rpy">
+  <xacro:macro name="box_inertia" params="m x y z o_xyz o_rpy">
     <inertial>
       <mass value="${m}" />
@@ -15,4 +15,4 @@
                 izz="${(m/12) * (y*y + y*y)}" />
     </inertial>
-  </xacro:xacro>
+  </xacro:macro>
 </robot>

File: src/robot_description/urdf/mobile_base.xacro (robot description, xacro)
@@ -20,4 +20,5 @@
       <material name="blue" />
     </visual>
+    <xacro:box_inertia m="5.0" x="${base_length}" y="${base_width}" z="${base_height}" o_xyz="0 0 ${base_height / 2}" o_rpy="0 0 0" />
   </link>
   <xacro:macro name="wheel_link" params="prefix">

Commit message: wheel inertia applied

File: src/robot_description/urdf/common_properties.xacro (robot description, xacro)
@@ -16,3 +16,21 @@
     </inertial>
   </xacro:macro>
+  <xacro:macro name="sphere_inertia" params="m r o_xyz o_rpy">
+    <inertial>
+      <mass value="${m}" />
+      <origin xyz="${o_xyz}" rpy="${o_rpy}" />
+      <inertia ixx="${(2.0/5.0)*m*r*r}" ixy="0" ixz="0"
+              iyy="${(2.0/5.0)*m*r*r}" iyz="0"
+              izz="${(2.0/5.0)*m*r*r}" />
+    </inertial>
+  </xacro:macro>
+  <xacro:macro name="cylinder_inertia" params="m r l o_xyz o_rpy">
+    <inertial>
+      <mass value="${m}" />
+      <origin xyz="${o_xyz}" rpy="${o_rpy}" />
+      <inertia  ixx="${(m/12) * (3*r*r + l*l)}" ixy="0" ixz="0"
+                iyy="${(m/12) * (3*r*r + l*l)}"            iyz="0"
+                izz="${(m/2) * (r*r)}" />
+    </inertial>
+  </xacro:macro>
 </robot>

File: src/robot_description/urdf/mobile_base.xacro (robot description, xacro)
@@ -31,4 +31,5 @@
         <material name="grey" />
       </visual>
+       <xacro:cylinder_inertia m="1.0" r="${wheel_radius}" l="${wheel_length}" o_xyz="0 0 0" o_rpy="${pi / 2.0} 0 0" />
     </link>
   </xacro:macro>
@@ -55,4 +56,5 @@
       <material name="grey" />
     </visual>
+    <xacro:sphere_inertia m="0.5" r="${wheel_radius / 2}" o_xyz="0 0 0" o_rpy="0 0 0" />
   </link>
   <joint name="base_caster_wheel_joint" type="fixed">

Commit message: robot bringup package with launch file

File: src/robot_description/urdf/common_properties.xacro (robot description, xacro)
@@ -20,7 +20,7 @@
       <mass value="${m}" />
       <origin xyz="${o_xyz}" rpy="${o_rpy}" />
-      <inertia ixx="${(2.0/5.0)*m*r*r}" ixy="0" ixz="0"
-              iyy="${(2.0/5.0)*m*r*r}" iyz="0"
-              izz="${(2.0/5.0)*m*r*r}" />
+      <inertia ixx="${(2.0/5.0)*m*r*r}"  ixy="0" ixz="0"
+               iyy="${(2.0/5.0)*m*r*r}"  iyz="0"
+               izz="${(2.0/5.0)*m*r*r}" />
     </inertial>
   </xacro:macro>
@@ -30,5 +30,5 @@
       <origin xyz="${o_xyz}" rpy="${o_rpy}" />
       <inertia  ixx="${(m/12) * (3*r*r + l*l)}" ixy="0" ixz="0"
-                iyy="${(m/12) * (3*r*r + l*l)}"            iyz="0"
+                iyy="${(m/12) * (3*r*r + l*l)}" iyz="0"
                 izz="${(m/2) * (r*r)}" />
     </inertial>

File: src/robot_description/urdf/mobile_base.xacro (robot description, xacro)
@@ -20,5 +20,12 @@
       <material name="blue" />
     </visual>
-    <xacro:box_inertia m="5.0" x="${base_length}" y="${base_width}" z="${base_height}" o_xyz="0 0 ${base_height / 2}" o_rpy="0 0 0" />
+    <xacro:box_inertia  m="5.0" x="${base_length}" y="${base_width}" z="${base_height}"
+                        o_xyz="0 0 ${base_height / 2}" o_rpy="0 0 0" />
+    <collision>
+      <geometry>
+        <box size="${base_length} ${base_width} ${base_height}" />
+      </geometry>
+      <origin xyz="0 0 ${base_height / 2}" rpy="0 0 0" />
+    </collision>
   </link>
   <xacro:macro name="wheel_link" params="prefix">
@@ -31,5 +38,12 @@
         <material name="grey" />
       </visual>
-       <xacro:cylinder_inertia m="1.0" r="${wheel_radius}" l="${wheel_length}" o_xyz="0 0 0" o_rpy="${pi / 2.0} 0 0" />
+      <collision>
+        <geometry>
+          <sphere radius="${wheel_radius}" length="${wheel_length}" />
+        </geometry>
+        <origin xyz="0 0 0" rpy="0 0 0" />
+      </collision>
+       <xacro:cylinder_inertia  m="1.0" r="${wheel_radius}" l="${wheel_length}"
+                                o_xyz="0 0 0" o_rpy="${pi / 2.0} 0 0" />
     </link>
   </xacro:macro>
@@ -56,4 +70,10 @@
       <material name="grey" />
     </visual>
+    <collision>
+      <geometry>
+        <sphere radius="${wheel_radius / 2}" />
+      </geometry>
+      <origin xyz="0 0 0" rpy="0 0 0" />
+    </collision>
     <xacro:sphere_inertia m="0.5" r="${wheel_radius / 2}" o_xyz="0 0 0" o_rpy="0 0 0" />
   </link>
