Commit message: sim time param and removed unused length param

File: src/robot_description/urdf/mobile_base.xacro (robot description, xacro)
@@ -40,5 +40,5 @@
       <collision>
         <geometry>
-          <sphere radius="${wheel_radius}" length="${wheel_length}" />
+          <sphere radius="${wheel_radius}" />
         </geometry>
         <origin xyz="0 0 0" rpy="0 0 0" />
