Commit message: rerouted lidar frme for gazebo

File: src/robot_description/urdf/lidar.xacro (robot description, xacro)
@@ -27,4 +27,10 @@
     <child link="lidar_link"/>
     <origin xyz="0 0 0.3" rpy="0 0 0"/>
+  </joint>
+  <link name="lidar_link_optical" />
+  <joint name="lidar_optical_joint" type="fixed">
+    <origin xyz="0 0 0" rpy="${-pi/2} 0 ${-pi/2}"/>
+    <parent link="lidar_link"/>
+    <child link="lidar_link_optical"/>
   </joint>
   <gazebo reference="lidar_link">

Commit message: rtbamap with lidar

File: src/robot_description/urdf/lidar.xacro (robot description, xacro)
@@ -8,5 +8,5 @@
         <cylinder radius="${lidar_radius}" length="${lidar_length}" />
       </geometry>
-      <material name="black" />
+      <material name="grey" />
     </visual>
     <collision>

Commit message: IMU link

File: src/robot_description/urdf/lidar.xacro (robot description, xacro)
@@ -1,65 +1,28 @@
 <?xml version="1.0"?>
 <robot xmlns:xacro="http://www.ros.org/wiki/xacro">
-  <xacro:property name="lidar_radius" value="0.05" />
-  <xacro:property name="lidar_length" value="0.05" />
-  <link name="lidar_link">
-    <visual>
-      <geometry>
-        <cylinder radius="${lidar_radius}" length="${lidar_length}" />
-      </geometry>
-      <material name="grey" />
-    </visual>
-    <collision>
-      <geometry>
-        <cylinder radius="${lidar_radius}" length="${lidar_length}" />
-      </geometry>
-    </collision>
-    <inertial>
-      <mass value="0.2"/>
-      <origin xyz="0 0 0" rpy="0 0 0"/>
-      <inertia ixx="0.001" ixy="0.0" ixz="0.0"
-              iyy="0.001" iyz="0.0"
-              izz="0.001"/>
-    </inertial>
-  </link>
-  <joint name="lidar_joint" type="fixed">
-    <parent link="base_link"/>
-    <child link="lidar_link"/>
-    <origin xyz="0 0 0.3" rpy="0 0 0"/>
-  </joint>
-  <link name="lidar_link_optical" />
-  <joint name="lidar_optical_joint" type="fixed">
-    <origin xyz="0 0 0" rpy="${-pi/2} 0 ${-pi/2}"/>
-    <parent link="lidar_link"/>
-    <child link="lidar_link_optical"/>
-  </joint>
-  <gazebo reference="lidar_link">
-    <sensor name="lidar" type="gpu_lidar">
-      <pose>0 0 0 0 0 0</pose>
-      <update_rate>20</update_rate>
-      <gz_frame_id>lidar_link</gz_frame_id>
-      <ray>
-        <scan>
-          <horizontal>
-            <samples>640</samples>
-            <resolution>1</resolution>
-            <min_angle>-3.14</min_angle>
-            <max_angle>3.14</max_angle>
-          </horizontal>
-          <vertical>
-            <samples>16</samples>
-            <resolution>1</resolution>
-            <min_angle>-0.26</min_angle>
-            <max_angle>0.26</max_angle>
-          </vertical>
-        </scan>
-        <range>
-          <min>0.08</min>
-          <max>30.0</max>
-          <resolution>0.01</resolution>
-        </range>
-      </ray>
-      <visualize>true</visualize>
-    </sensor>
-  </gazebo>
+  <xacro:macro name="imu_sensor_macro" params="parent_link">
+    <!-- IMU Link -->
+    <link name="imu_link">
+      <inertial>
+        <origin xyz="0 0 0" rpy="0 0 0"/>
+        <mass value="0.1"/>
+        <inertia ixx="1e-5" ixy="0" ixz="0" iyy="1e-5" iyz="0" izz="1e-5"/>
+      </inertial>
+    </link>
+    <!-- Fixed Joint between base and IMU -->
+    <joint name="imu_joint" type="fixed">
+      <parent link="${parent_link}"/>
+      <child link="imu_link"/>
+      <origin xyz="0 0 0" rpy="0 0 0"/> <!-- adjust if you want to offset the IMU -->
+    </joint>
+    <!-- Gazebo IMU Plugin -->
+    <gazebo>
+      <plugin name="imu_plugin" filename="gz-sim-imu-system">
+        <topic>imu/data</topic>
+        <frame_id>imu_link</frame_id>
+        <gaussian_noise>0.01</gaussian_noise>
+        <update_rate>50.0</update_rate>
+      </plugin>
+    </gazebo>
+  </xacro:macro>
 </robot>

File: src/robot_description/urdf/robot.urdf.xacro (robot description, xacro)
@@ -6,3 +6,5 @@
   <xacro:include filename="camera.xacro" />
   <xacro:include filename="lidar.xacro" />
+  <xacro:include filename="IMU.xacro" />
+  <xacro:imu_sensor_macro parent_link="base_link"/>
 </robot>

Commit message: ammended lidar

File: src/robot_description/urdf/lidar.xacro (robot description, xacro)
@@ -1,28 +1,65 @@
 <?xml version="1.0"?>
 <robot xmlns:xacro="http://www.ros.org/wiki/xacro">
-  <xacro:macro name="imu_sensor_macro" params="parent_link">
-    <!-- IMU Link -->
-    <link name="imu_link">
-      <inertial>
-        <origin xyz="0 0 0" rpy="0 0 0"/>
-        <mass value="0.1"/>
-        <inertia ixx="1e-5" ixy="0" ixz="0" iyy="1e-5" iyz="0" izz="1e-5"/>
-      </inertial>
-    </link>
-    <!-- Fixed Joint between base and IMU -->
-    <joint name="imu_joint" type="fixed">
-      <parent link="${parent_link}"/>
-      <child link="imu_link"/>
-      <origin xyz="0 0 0" rpy="0 0 0"/> <!-- adjust if you want to offset the IMU -->
-    </joint>
-    <!-- Gazebo IMU Plugin -->
-    <gazebo>
-      <plugin name="imu_plugin" filename="gz-sim-imu-system">
-        <topic>imu/data</topic>
-        <frame_id>imu_link</frame_id>
-        <gaussian_noise>0.01</gaussian_noise>
-        <update_rate>50.0</update_rate>
-      </plugin>
-    </gazebo>
-  </xacro:macro>
+  <xacro:property name="lidar_radius" value="0.05" />
+  <xacro:property name="lidar_length" value="0.05" />
+  <link name="lidar_link">
+    <visual>
+      <geometry>
+        <cylinder radius="${lidar_radius}" length="${lidar_length}" />
+      </geometry>
+      <material name="grey" />
+    </visual>
+    <collision>
+      <geometry>
+        <cylinder radius="${lidar_radius}" length="${lidar_length}" />
+      </geometry>
+    </collision>
+    <inertial>
+      <mass value="0.2"/>
+      <origin xyz="0 0 0" rpy="0 0 0"/>
+      <inertia ixx="0.001" ixy="0.0" ixz="0.0"
+              iyy="0.001" iyz="0.0"
+              izz="0.001"/>
+    </inertial>
+  </link>
+  <joint name="lidar_joint" type="fixed">
+    <parent link="base_link"/>
+    <child link="lidar_link"/>
+    <origin xyz="0 0 0.3" rpy="0 0 0"/>
+  </joint>
+  <link name="lidar_link_optical" />
+  <joint name="lidar_optical_joint" type="fixed">
+    <origin xyz="0 0 0" rpy="${-pi/2} 0 ${-pi/2}"/>
+    <parent link="lidar_link"/>
+    <child link="lidar_link_optical"/>
+  </joint>
+  <gazebo reference="lidar_link">
+    <sensor name="lidar" type="gpu_lidar">
+      <pose>0 0 0 0 0 0</pose>
+      <update_rate>20</update_rate>
+      <gz_frame_id>lidar_link</gz_frame_id>
+      <ray>
+        <scan>
+          <horizontal>
+            <samples>640</samples>
+            <resolution>1</resolution>
+            <min_angle>-3.14</min_angle>
+            <max_angle>3.14</max_angle>
+          </horizontal>
+          <vertical>
+            <samples>16</samples>
+            <resolution>1</resolution>
+            <min_angle>-0.26</min_angle>
+            <max_angle>0.26</max_angle>
+          </vertical>
+        </scan>
+        <range>
+          <min>0.08</min>
+          <max>30.0</max>
+          <resolution>0.01</resolution>
+        </range>
+      </ray>
+      <visualize>true</visualize>
+    </sensor>
+  </gazebo>
 </robot>
