Commit message: revised IMU

File: src/robot_description/urdf/IMU.xacro (robot description, xacro)
@@ -2,23 +2,23 @@
 <robot xmlns:xacro="http://www.ros.org/wiki/xacro">
   <xacro:macro name="imu_sensor_macro" params="parent_link">
-  <link name="imu_link">
-    <inertial>
-      <mass value="0.1"/>
-      <origin xyz="0 0 0" rpy="0 0 0"/>
-      <inertia ixx="1e-5" ixy="0" ixz="0" iyy="1e-5" iyz="0" izz="1e-5"/>
-    </inertial>
-  </link>
-  <joint name="imu_joint" type="fixed">
-    <parent link="${parent_link}"/>
-    <child link="imu_link"/>
-  </joint>
-  <gazebo>
-    <plugin name="gz::sim::systems::Imu" filename="gz-sim-imu-system">
-      <topic>imu/data</topic>
-      <frame_id>imu_link</frame_id>
-      <gaussian_noise>0.01</gaussian_noise>
-      <update_rate>50.0</update_rate>
-    </plugin>
-  </gazebo>
-</xacro:macro>
+    <link name="imu_link">
+      <inertial>
+        <mass value="0.1"/>
+        <origin xyz="0 0 0" rpy="0 0 0"/>
+        <inertia ixx="1e-5" ixy="0" ixz="0" iyy="1e-5" iyz="0" izz="1e-5"/>
+      </inertial>
+      <gazebo>
+        <plugin name="gz::sim::systems::Imu" filename="gz-sim-imu-system">
+          <topic>imu/data</topic>
+          <frame_id>imu_link</frame_id>
+          <gaussian_noise>0.01</gaussian_noise>
+          <update_rate>50.0</update_rate>
+        </plugin>
+      </gazebo>
+    </link>
+    <joint name="imu_joint" type="fixed">
+      <parent link="${parent_link}"/>
+      <child link="imu_link"/>
+    </joint>
+  </xacro:macro>
 </robot>

Commit message: imu topic streaming

File: src/robot_description/urdf/IMU.xacro (robot description, xacro)
@@ -1,24 +1,20 @@
 <?xml version="1.0"?>
 <robot xmlns:xacro="http://www.ros.org/wiki/xacro">
-  <xacro:macro name="imu_sensor_macro" params="parent_link">
-    <link name="imu_link">
-      <inertial>
-        <mass value="0.1"/>
-        <origin xyz="0 0 0" rpy="0 0 0"/>
-        <inertia ixx="1e-5" ixy="0" ixz="0" iyy="1e-5" iyz="0" izz="1e-5"/>
-      </inertial>
-      <gazebo>
-        <plugin name="gz::sim::systems::Imu" filename="gz-sim-imu-system">
-          <topic>imu/data</topic>
-          <frame_id>imu_link</frame_id>
-          <gaussian_noise>0.01</gaussian_noise>
-          <update_rate>50.0</update_rate>
-        </plugin>
-      </gazebo>
-    </link>
-    <joint name="imu_joint" type="fixed">
-      <parent link="${parent_link}"/>
-      <child link="imu_link"/>
-    </joint>
-  </xacro:macro>
+  <joint name="imu_joint" type="fixed">
+    <origin xyz="0 0 0" rpy="0 0 0" />
+    <parent link="base_link"/>
+    <child link="imu_link" />
+  </joint>
+  <link name="imu_link">
+  </link>
+  <gazebo reference="imu_link">
+    <sensor name="imu" type="imu">
+      <always_on>1</always_on>
+      <update_rate>50</update_rate>
+      <visualize>true</visualize>
+      <topic>imu</topic>
+      <enable_metrics>true</enable_metrics>
+      <gz_frame_id>imu_link</gz_frame_id>
+    </sensor>
+  </gazebo>
 </robot>

File: src/robot_description/urdf/robot.urdf.xacro (robot description, xacro)
@@ -7,4 +7,3 @@
   <xacro:include filename="lidar.xacro" />
   <xacro:include filename="IMU.xacro" />
-  <xacro:imu_sensor_macro parent_link="base_link"/>
 </robot>
