Commit message: lidar2d lidar3d setup

File: src/yahboom_rosmaster/yahboom_rosmaster_description/urdf/robots/rosmaster_x3.urdf.xacro (robot description, xacro)
@@ -8,5 +8,6 @@
     <xacro:include filename="$(find yahboom_rosmaster_description)/urdf/mech/mecanum_wheel.urdf.xacro"/>
     <xacro:include filename="$(find yahboom_rosmaster_description)/urdf/sensors/rgbd_camera.urdf.xacro"/>
-    <xacro:include filename="$(find yahboom_rosmaster_description)/urdf/sensors/lidar.urdf.xacro"/>
+    <xacro:include filename="$(find yahboom_rosmaster_description)/urdf/sensors/lidar2D.urdf.xacro"/>
+    <xacro:include filename="$(find yahboom_rosmaster_description)/urdf/sensors/lidar3D.urdf.xacro"/>
     <xacro:include filename="$(find yahboom_rosmaster_description)/urdf/sensors/imu.urdf.xacro"/>
     <xacro:rosmaster_x3_base prefix="$(arg prefix)"/>
@@ -36,5 +37,5 @@
       xyz_offset="0.105 0 0.05"
       rpy_offset="0 -0.50 0"/>
-    <xacro:lidar_sensor
+    <xacro:lidar2D_sensor
       prefix="$(arg prefix)"
       parent="base_link"
@@ -45,4 +46,13 @@
       mesh_rpy_offset="${-M_PI/2} 0 0"
       topic_name="scan"/>
+    <xacro:lidar3D_sensor
+      prefix="$(arg prefix)"
+      parent="base_link"
+      frame_id="lidar3d_frame"
+      xyz_offset="0 0 0.0825"
+      rpy_offset="0 0 0"
+      mesh_xyz_offset="0 0 0"
+      mesh_rpy_offset="${-M_PI/2} 0 0"
+      topic_name="lidar/points/points"/>
     <xacro:imu_sensor
       prefix="$(arg prefix)"

File: src/yahboom_rosmaster/yahboom_rosmaster_description/urdf/sensors/lidar2D.urdf.xacro (robot description, xacro)
@@ -2,5 +2,5 @@
 <robot xmlns:xacro="http://www.ros.org/wiki/xacro">
   <xacro:property name="M_PI" value="3.1415926535897931" />
-  <xacro:macro name="lidar_sensor" params="
+  <xacro:macro name="lidar2D_sensor" params="
     prefix:=''
     parent:='base_link'
@@ -79,5 +79,6 @@
         <specular>${gazebo_material_specular}</specular>
       </material>
-      <!-- <sensor name="${prefix}lidar_sensor" type="gpu_lidar">
+      <!-- 2D LIDAR -->
+      <sensor name="${prefix}lidar2D_sensor" type="gpu_lidar">
         <topic>${topic_name}</topic>
         <update_rate>${update_rate}</update_rate>
@@ -106,35 +107,5 @@
         </ray>
         <gz_frame_id>${prefix}${frame_id}</gz_frame_id>
-      </sensor> -->
-        <sensor name="${prefix}lidar_sensor" type="gpu_lidar">
-          <topic>${topic_name}</topic>
-          <!-- <pose>0 0 0 0 0 0</pose> -->
-          <update_rate>${update_rate}</update_rate>
-          <always_on>${always_on}</always_on>
-          <gz_frame_id>${prefix}${frame_id}</gz_frame_id>
-          <visualize>${visualize}</visualize>
-          <ray>
-            <scan>
-              <horizontal>
-                <samples>640</samples>
-                <resolution>1</resolution>
-                <min_angle>-3.14</min_angle>
-                <max_angle>3.14</max_angle>
-              </horizontal>
-              <vertical>
-                <samples>16</samples>
-                <resolution>1</resolution>
-                <min_angle>-0.26</min_angle>
-                <max_angle>0.26</max_angle>
-              </vertical>
-            </scan>
-            <range>
-              <min>0.08</min>
-              <max>30.0</max>
-              <resolution>0.01</resolution>
-            </range>
-          </ray>
-          <visualize>true</visualize>
-        </sensor>
+      </sensor>
     </gazebo>
   </xacro:macro>
