Commit message: first robot camera mesh visibility off and rviz config

File: src/first_robot/robot_description/urdf/camera.xacro (robot description, xacro)
@@ -5,10 +5,10 @@
     <xacro:property name="camera_height" value="0.05" />
     <link name="camera_link">
-        <visual>
+        <!-- <visual>
             <geometry>
                 <box size="${camera_length} ${camera_width} ${camera_height}" />
             </geometry>
             <material name="grey" />
-        </visual>
+        </visual> -->
         <collision>
             <geometry>
@@ -22,5 +22,5 @@
         <parent link="base_link" />
         <child link="camera_link" />
-        <origin xyz="${(base_length + camera_length) / 2.0} 0 ${base_height / 2.0}" rpy="0 0 0" />
+        <origin xyz="${(base_length + camera_length) / 2.0} 0 ${base_height * 2.0}" rpy="0 0 0" />
     </joint>
     <link name="camera_link_optical" />

File: src/first_robot/robot_description/urdf/robot.urdf.xacro (robot description, xacro)
@@ -5,5 +5,5 @@
   <xacro:include filename="mobile_base_gazebo.xacro" />
   <xacro:include filename="camera.xacro" />
-  <xacro:include filename="lidar.xacro" />
+  <!-- <xacro:include filename="lidar.xacro" /> -->
   <xacro:include filename="IMU.xacro" />
 </robot>
